File: ws2812b_ctrl_RF.kicad_pcb (KiCad board)
At the start: 2 copper layers, 65 x 65 mm, 42 parts, among them K1 SANYOU_SRD_Form_C, Q1 Q_PNP_BEC, Q2 Q_NPN_BEC, U1 4081, U2 74HC02, U3 AMS1117-3.3

Commit message: Version 2.
Parts:
- removed C1, C13: CP, Capacitor_Tantalum_SMD:CP_EIA-3216-12_Kemet-S
- removed CTL1: CONN_01, Connectors:1X01
- removed FB2: Ferrite_Bead, Inductor_SMD:L_1210_3225Metric
- added D2: ZMMxx, Diode_SMD:D_MiniMELF_Handsoldering, B.Cu at (81.8, 90.9)
- added DBG1: LED, LED_SMD:LED_1206_3216Metric, F.Cu at (104.1, 130.9)
- added F1: Fuse_Polarized, Fuse:Fuse_1812_4532Metric_Pad1.30x3.40mm_HandSolder, B.Cu at (76.5, 91.2)
- added J1: Conn_01x03_Female, Connector_JST:JST_XH_B3B-XH-A_1x03_P2.50mm_Vertical, F.Cu at (73.9, 81.8)
- added J2: Conn_01x04_Female, Connector_JST:JST_XH_B4B-XH-A_1x04_P2.50mm_Vertical, F.Cu at (124.7, 73.9)
- added J3: Conn_01x01_Male, Connector_Pin:Pin_D1.0mm_L10.0mm, F.Cu at (97.0, 128.8)
- added Q3: NPN BC817, Package_TO_SOT_SMD:SOT-23, F.Cu at (106.1, 125.7)
- added Q4: IRLML5203, Package_TO_SOT_SMD:SOT-23, B.Cu at (86.6, 97.3)
- added R1: 560, Resistors:0805, F.Cu at (112.8, 129.7)
- added R10: 4K7, Resistors:0805, F.Cu at (106.2, 129.1)
- added R11: 560, Resistors:0805, F.Cu at (109.0, 123.6)
- added R12: 470K, Resistors:0805, F.Cu at (106.2, 122.9)
- added R13: 10K, Resistors:0805, B.Cu at (107.3, 84.8)
- added R14: 470k, Resistors:0805, B.Cu at (86.5, 100.1)
- added R15: 470K, Resistors:0805, F.Cu at (114.8, 126.2)
- added R16: 33, Resistors:0805, B.Cu at (89.8, 100.1)
- added R9: 4K7, Resistors:0805, B.Cu at (85.2, 115.1)
- B1: value ARDUINO_PRO_MINI -> ARDUINO_PRO_MINI_SIMPLE; footprint Boards:ARDUINO_PRO_MINI_SIMPLE -> Boards:ARDUINO_PRO_MINI
- C10, C12, C2, C4, C6: value C -> 100nF
- C11: value CP -> 10uF; footprint Capacitor_Tantalum_SMD:CP_EIA-3216-12_Kemet-S -> Capacitor_Tantalum_SMD:CP_EIA-3528-21_Kemet-B_Pad1.50x2.35mm_HandSolder
- C5, C8: footprint Capacitor_Tantalum_SMD:CP_EIA-3216-12_Kemet-S -> Capacitor_Tantalum_SMD:CP_EIA-3528-21_Kemet-B_Pad1.50x2.35mm_HandSolder
- C9: value CP -> 22uF; footprint Capacitor_Tantalum_SMD:CP_EIA-3216-12_Kemet-S -> Capacitor_Tantalum_SMD:CP_EIA-3528-21_Kemet-B_Pad1.50x2.35mm_HandSolder
- D1: value D -> SS14
- ISP1: footprint Connector_PinHeader_2.54mm:PinHeader_2x03_P2.54mm_Vertical -> Connector_IDC:IDC-Header_2x03_P2.54mm_Vertical
- Q1: value Q_PNP_BEC -> PNP BC807
- Q2: value Q_NPN_BEC -> NPN BC817
- R17: renamed from R1; value R -> 100K; moved to B.Cu
- R2, R7: value R -> 470K
- R3: value R -> 4K7
- R5: value R -> 200
- R6: value R -> 330
- R8: value R -> 560
- RLY1: renamed from XnRF1; moved to F.Cu
- moved C5 28.3 mm to (79.8, 82.0), turned to 0 degrees
- moved ~SS1 25.5 mm to (110.0, 130.8), turned to 90 degrees
- moved Q1 25.2 mm to (111.7, 126.2)
- moved R3 25.1 mm to (108.0, 129.2)
- moved R17 14.0 mm to (107.3, 88.1), turned to 0 degrees
- moved C8 10.4 mm to (85.1, 82.0), turned to 180 degrees
- moved RLY1 9.52 mm to (73.2, 114.6), turned to 270 degrees
- moved FB1 9.41 mm to (83.1, 98.4)
- moved RS485 7.75 mm to (80.5, 74.4), turned to 0 degrees
- moved SUPPLY1 7.12 mm to (74.2, 100.6)
- moved ISP1 5.95 mm to (126.2, 90.7)
- moved C11 4.40 mm to (93.5, 92.6)
- moved C12 3.49 mm to (79.4, 78.0), turned to 0 degrees
- moved U3 1.53 mm to (87.4, 90.9)
- moved C9 0.96 mm to (90.9, 80.6), turned to 270 degrees
- renumbered XnRF2 to ~SS1
Connections:
- B1 pad 10: (no net) -> /Vsup
- B1 pad 11: (no net) -> /RLYCTL
- B1 pad 12: (no net) -> /V33CTL
- B1 pad 17: /RLYCTL -> /nRFIRQ
- B1 pad 19: /nRFIRQ -> /Vsup
- B1 pad 20: (no net) -> /ExtADC
- B1 pad 5: (no net) -> /INT0
- B1 pad 7: (no net) -> /ExtIC
- B1 pad 8: (no net) -> /DBGCTL
- B1 pad 9: (no net) -> /ExtPWM
- C8 pad 1: VCC -> Net-(C8-Pad1)
- D1 pad 1: Net-(D1-Pad1) -> VCC
- FB1 pad 1: +5V -> Net-(D2-Pad1)
- FB1 pad 2: VCC -> +5V
- K1 pad 5: Net-(D1-Pad1) -> VCC
- Q1 pad 1: /~SS -> Net-(Q1-Pad1)
- R17 pad 1: +5V -> VCC
- R17 pad 2: /~SS -> /Vsup
- RLY1 pad 1: Net-(D1-Pad1) -> Net-(R9-Pad1)
- U3 pad 2: Net-(FB2-Pad2) -> /3.3V
- U3 pad 3: VCC -> Net-(C8-Pad1)
Routing:
- net GND: track 290.1 -> 364.4 mm, vias 2 -> 5
- net VCC: track 41.7 -> 86.8 mm, vias 0 -> 2
- net /DBGCTL: track 0.00 -> 39.8 mm
- net /ExtPWM: track 0.00 -> 37.6 mm
- net /ExtIC: track 0.00 -> 29.9 mm
- net /~SS: track 32.8 -> 59.5 mm
- net /Vsup: track 0.00 -> 24.3 mm
- net /INT0: track 0.00 -> 24.0 mm
- net Net-(C8-Pad1): track 0.00 -> 17.3 mm
- net /ExtADC: track 0.00 -> 16.4 mm
- net /RLYCTL: track 30.3 -> 16.3 mm
- net Net-(R9-Pad1): track 0.00 -> 12.0 mm, vias 0 -> 1
- net Net-(FB2-Pad2): track 11.2 -> 0.00 mm
- net Net-(D2-Pad1): track 0.00 -> 8.03 mm
- net Net-(D1-Pad1): track 7.70 -> 0.00 mm
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