File: ws2812b_ctrl_RF.sch (KiCad schematic (older format))
At the start: 42 parts, among them K1 SANYOU_SRD_Form_C, Q1 Q_PNP_BEC, Q2 Q_NPN_BEC, U1 4081, U2 74HC02, U3 AMS1117-3.3

Commit message: Version 2.
Parts:
- removed C1, C13: CP, Capacitor_Tantalum_SMD:CP_EIA-3216-12_Kemet-S, symbol Device:CP
- removed CTL1: CONN_01, Connectors:1X01, symbol SparkFun-Connectors:CONN_01
- removed FB2: Ferrite_Bead, Inductor_SMD:L_1210_3225Metric, symbol Device:Ferrite_Bead
- added D2: ZMMxx, Diode_SMD:D_MiniMELF_Handsoldering, symbol Diode:ZMMxx
- added DBG1: LED, LED_SMD:LED_1206_3216Metric, symbol Device:LED
- added F1: Fuse_Polarized, Fuse:Fuse_1812_4532Metric_Pad1.30x3.40mm_HandSolder, symbol Device:Fuse_Polarized
- added J1: Conn_01x03_Female, Connector_JST:JST_XH_B3B-XH-A_1x03_P2.50mm_Vertical, symbol Connector:Conn_01x03_Female
- added J2: Conn_01x04_Female, Connector_JST:JST_XH_B4B-XH-A_1x04_P2.50mm_Vertical, symbol Connector:Conn_01x04_Female
- added J3: Conn_01x01_Male, Connector_Pin:Pin_D1.0mm_L10.0mm, symbol Connector:Conn_01x01_Male
- added Q3: NPN BC817, Package_TO_SOT_SMD:SOT-23, symbol Device:Q_NPN_BEC
- added Q4: IRLML5203, Package_TO_SOT_SMD:SOT-23, symbol Transistor_FET:IRLML5203
- added R1, R11: 560, Resistors:0805, symbol Device:R
- added R10, R9: 4K7, Resistors:0805, symbol Device:R
- added R12, R15: 470K, Resistors:0805, symbol Device:R
- added R13: 10K, Resistors:0805, symbol Device:R
- added R14: 470k, Resistors:0805, symbol Device:R
- added R16: 33, Resistors:0805, symbol Device:R
- B1: value ARDUINO_PRO_MINI -> ARDUINO_PRO_MINI_SIMPLE; footprint Boards:ARDUINO_PRO_MINI_SIMPLE -> Boards:ARDUINO_PRO_MINI
- C10, C12, C2, C4, C6: value C -> 100nF
- C11: value CP -> 10uF; footprint Capacitor_Tantalum_SMD:CP_EIA-3216-12_Kemet-S -> Capacitor_Tantalum_SMD:CP_EIA-3528-21_Kemet-B_Pad1.50x2.35mm_HandSolder
- C5, C8: footprint Capacitor_Tantalum_SMD:CP_EIA-3216-12_Kemet-S -> Capacitor_Tantalum_SMD:CP_EIA-3528-21_Kemet-B_Pad1.50x2.35mm_HandSolder
- C9: value CP -> 22uF; footprint Capacitor_Tantalum_SMD:CP_EIA-3216-12_Kemet-S -> Capacitor_Tantalum_SMD:CP_EIA-3528-21_Kemet-B_Pad1.50x2.35mm_HandSolder
- D1: value D -> SS14
- ISP1: footprint Connector_PinHeader_2.54mm:PinHeader_2x03_P2.54mm_Vertical -> Connector_IDC:IDC-Header_2x03_P2.54mm_Vertical
- Q1: value Q_PNP_BEC -> PNP BC807
- Q2: value Q_NPN_BEC -> NPN BC817
- R17: renamed from R1; value R -> 100K
- R2, R7: value R -> 470K
- R3: value R -> 4K7
- R5: value R -> 200
- R6: value R -> 330
- R8: value R -> 560
- renumbered XnRF1 to RLY1, XnRF2 to ~SS1
Connections:
- net labels added: DBGCTL, ExtADC, ExtIC, ExtPWM, INT0, V33CTL, Vsup
- wire segments 160 -> 208
Other:
- moved on the sheet: C10, C12, C2, C4, C8, FB1, H1, H2, H3, H4, R17, R5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

Commit message: Added HW v1 schematic and PCB layout images.
Parts:
- C5, C8: value CP -> 100uF
Changed lines of the file:
@@
 P 850 6550
 F 0 "C8" H 968 6596 50  0000 L CNN
-F 1 "CP" H 968 6505 50  0000 L CNN
+F 1 "100uF" H 968 6505 50  0000 L CNN
 F 2 "Capacitor_Tantalum_SMD:CP_EIA-3528-21_Kemet-B_Pad1.50x2.35mm_HandSolder" H 888 6400 50  0001 C CNN
 F 3 "~" H 850 6550 50  0001 C CNN
@@
 P 2800 2000
 F 0 "C5" H 2918 2046 50  0000 L CNN
-F 1 "CP" H 2918 1955 50  0000 L CNN
+F 1 "100uF" H 2918 1955 50  0000 L CNN
 F 2 "Capacitor_Tantalum_SMD:CP_EIA-3528-21_Kemet-B_Pad1.50x2.35mm_HandSolder" H 2838 1850 50  0001 C CNN
 F 3 "~" H 2800 2000 50  0001 C CNN
